File: CustomTKL101.sch (KiCad schematic (older format))
At the start: 10 parts

Commit message: 15-02-2020
Parts:
- removed C?: 1uF, symbol Device:C_Small
- removed C? (x2): 22pF, symbol Device:C_Small
- removed R? (x2): 10k, symbol Device:R_Small
- removed R? (x2): 22, symbol Device:R_Small
- removed SW?: SW_Push, symbol Switch:SW_Push
- removed U?: AT90USB1286-AU, Package_QFP:TQFP-64_14x14mm_P0.8mm, symbol MCU_Microchip_AVR:AT90USB1286-AU
- removed Y?: 16MHz, symbol Device:Crystal_GND24_Small
- added C?: 1uF, symbol Device:C_Small
- added C?: 10uF, symbol Device:C_Small
- added C? (x3): 0.1uF, symbol Device:C_Small
- added C? (x2): 22pF, symbol Device:C_Small
- added R? (x2): 10k, symbol Device:R_Small
- added R? (x2): 22, symbol Device:R_Small
- added SW?: SW_Push, symbol Switch:SW_Push
- added U?: ATmega32U4-AU, Package_QFP:TQFP-44_10x10mm_P0.8mm, symbol MCU_Microchip_ATmega:ATmega32U4-AU
- added Y?: 16MHz, symbol Device:Crystal_GND24_Small
Connections:
- net +5V: now also C?.1, C?.1, C?.1, C?.1, R?.1, U?.14 (VCC), U?.2 (UVCC), U?.24 (AVCC), U?.34 (VCC), U?.44 (AVCC), U?.7 (VBUS)
- net D+: now also R?.2
- net D-: now also R?.2
- net GND: now also C?.2, C?.2, C?.2, C?.2, C?.2, C?.2, C?.2, R?.1, SW?.1, U?.15 (GND), U?.23 (GND), U?.35 (GND), U?.43 (GND), U?.5 (UGND), Y?.2, Y?.4
- new net: R?.2, SW?.2, U?.13 (~RESET)
- new net: C?.1, U?.16 (XTAL2), Y?.3
- new net: C?.1, U?.17 (XTAL1), Y?.1
- new net: R?.1, U?.3 (D-)
- new net: R?.2, U?.33 (~HWB~/PE2)
- new net: R?.1, U?.4 (D+)
- new net: C?.1, U?.6 (UCAP)

Commit message: Schematic Progress
Parts:
- added D? (x126): D_Small, symbol Device:D_Small
- added F?: 500mA, symbol Device:Polyfuse_Small
- added J?: USB4085-GF-A_REVA, GCT_USB4085-GF-A_REVA, symbol USB4085-GF-A_REVA:USB4085-GF-A_REVA
- added MX? (x126): MX-NoLED, symbol MX_Alps_Hybrid:MX-NoLED
- added R? (x4): 5.1kohm, symbol Device:R_Small
- added R?: 1.5k, symbol Device:R_Small
Connections:
- net labels added: DB+, DB-
- wire segments 47 -> 588
Other:
- moved on the sheet: C?, R?, SW?, U?, Y?

Commit message: Progress on Schematic
Parts:
- removed D? (x25): D_Small, symbol Device:D_Small
- removed MX? (x25): MX-NoLED, symbol MX_Alps_Hybrid:MX-NoLED
Connections:
- net labels added: Col0&1, Col10&11, Col12&13, Col14&15, Col16&17, Col18&19, Col2&3, Col20, Col4&5, Col6&7, Col8&9, Row0.1, Row0.2, Row1.1, Row1.2, Row2.1, Row2.2, Row3.1, Row3.2, Row4.1, Row4.2, Row5.1, Row5.2
- wire segments 588 -> 512
