File: CustomTKL101.kicad_pcb (KiCad board)
At the start: 2 copper layers, 422.3 x 131.8 mm, 220 parts, among them J1 USB4085-GF-A_REVA, SW1 SW_Push, U1 ATmega32U4-AU, Y1 16MHz

Commit message: Completed PCB ?
Parts:
- MX101, MX32: footprint MX_Alps_Hybrid:MX-1U-NoLED -> MX_Alps_Hybrid:MX-2U-ReversedStabilizers-NoLED
- MX71, MX75: footprint MX_Alps_Hybrid:MX-1U-NoLED -> MX_Alps_Hybrid:MX-2.25U-ReversedStabilizers-NoLED
- MX86: footprint MX_Alps_Hybrid:MX-1U-NoLED -> MX_Alps_Hybrid:MX-2.75U-ReversedStabilizers-NoLED
- MX93: footprint MX_Alps_Hybrid:MX-1U-NoLED -> MX_Alps_Hybrid:MX-6.25U-ReversedStabilizers-NoLED
Connections:
- U1 pad 10: Col6&7 -> Col16&17
- U1 pad 11: Col8&9 -> Col14&15
- U1 pad 12: Col10&11 -> Net-(U1-Pad12)
- U1 pad 18: Col20 -> Col2&3
- U1 pad 19: Col18&19 -> Col4&5
- U1 pad 20: Col16&17 -> Col6&7
- U1 pad 21: Col14&15 -> Col8&9
- U1 pad 22: Col12&13 -> Col10&11
- U1 pad 27: Net-(U1-Pad27) -> Col12&13
- U1 pad 8: Col2&3 -> Col20
- U1 pad 9: Col4&5 -> Col18&19
Routing:
- net Col20: track 485.3 -> 456.9 mm
- net Col8&9: track 395.3 -> 376.2 mm, vias 1 -> 4
- net Col10&11: track 410.4 -> 393.3 mm, vias 1 -> 4
- net Col6&7: track 334.4 -> 317.8 mm, vias 1 -> 4
- net Col4&5: track 317.6 -> 301.2 mm, vias 1 -> 4
- net GND: track 148.8 -> 137.7 mm
- net Col14&15: track 475.8 -> 465.5 mm, vias 1 -> 4
- net Col2&3: track 179.0 -> 169.0 mm, vias 1 -> 4
- net Col12&13: track 436.9 -> 430.6 mm, vias 3 -> 4
- net +5V: track 106.9 -> 102.9 mm
- net Col18&19: track 582.7 -> 578.9 mm, vias 1 -> 4
- net Col16&17: track 588.6 -> 586.1 mm, vias 3 -> 4
- net D+: track 27.9 -> 29.9 mm
- net Row2.2: track 404.4 -> 406.2 mm
- net D-: track 29.7 -> 30.9 mm
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Other:
- net class Power added: clearance 0.2, trace_width 0.4, via_dia 0.8, via_drill 0.4

Commit message: Filled GND + Wiring fixes
Routing:
- net Col16&17: track 586.1 -> 570.7 mm
- net Row5.1: track 498.9 -> 501.3 mm
- net Col20: track 456.9 -> 457.5 mm
- added copper zone on B.Cu, net GND
- added copper zone on F.Cu, net GND
